Commit message: * mark II: new leg model

File: rex_gym/util/pybullet_data/assets/urdf/rex_arm.urdf (robot description, URDF)
Before this commit: robot rex_arm, 31 links, 30 joints
Links:
- link front_left_foot_link: geometry collision box size=0.026 0.020 0.115; visual mesh filename=stl/lower_leg_solid.stl scale=0.001 0.001 0.001
- link front_left_leg_link: geometry collision box size=0.028 0.036 0.12; visual mesh filename=stl/upper_leg_shell_base.stl scale=0.001 0.001 0.001
- link front_left_leg_link_cover: geometry visual mesh filename=stl/upper_leg_shell_cover.stl scale=0.001 0.001 0.001
- link front_right_foot_link: geometry collision box size=0.026 0.020 0.115; visual mesh filename=stl/lower_leg_solid.stl scale=0.001 0.001 0.001
- link front_right_leg_link: geometry collision box size=0.028 0.036 0.12; visual mesh filename=stl/upper_leg_shell_base.stl scale=0.001 0.001 0.001
- link front_right_leg_link_cover: geometry visual mesh filename=stl/upper_leg_shell_cover.stl scale=0.001 0.001 0.001
- link rear_left_foot_link: geometry collision box size=0.026 0.020 0.115; visual mesh filename=stl/lower_leg_solid.stl scale=0.001 0.001 0.001
- link rear_left_leg_link: geometry collision box size=0.028 0.036 0.12; visual mesh filename=stl/upper_leg_shell_base.stl scale=0.001 0.001 0.001
- link rear_left_leg_link_cover: geometry visual mesh filename=stl/upper_leg_shell_cover.stl scale=0.001 0.001 0.001
- link rear_right_foot_link: geometry collision box size=0.026 0.020 0.115; visual mesh filename=stl/lower_leg_solid.stl scale=0.001 0.001 0.001
- link rear_right_leg_link: geometry collision box size=0.028 0.036 0.12; visual mesh filename=stl/upper_leg_shell_base.stl scale=0.001 0.001 0.001
- link rear_right_leg_link_cover: geometry visual mesh filename=stl/upper_leg_shell_cover.stl scale=0.001 0.001 0.001
Joints:
- joint foot_motor_front_left: limit lower=-0.1 upper=2.59 effort=100.0 velocity=0.5 -> lower=-3.14 upper=3.14 effort=100.0 velocity=0.5; origin xyz=-0.01 0 -0.12 rpy=0 0 0 -> xyz=0.002 -0.02 -0.16 rpy=0 0 0
- joint foot_motor_front_right: limit lower=-0.1 upper=2.59 effort=100.0 velocity=0.5 -> lower=-3.14 upper=3.14 effort=100.0 velocity=0.5; origin xyz=-0.01 0 -0.12 rpy=0 0 0 -> xyz=0.002 0.02 -0.16 rpy=0 0 0
- joint foot_motor_rear_left: limit lower=-0.1 upper=2.59 effort=100.0 velocity=0.5 -> lower=-3.14 upper=3.14 effort=100.0 velocity=0.5; origin xyz=-0.01 0 -0.12 rpy=0 0 0 -> xyz=0.002 -0.02 -0.16 rpy=0 0 0
- joint foot_motor_rear_right: limit lower=-0.1 upper=2.59 effort=100.0 velocity=0.5 -> lower=-3.14 upper=3.14 effort=100.0 velocity=0.5; origin xyz=-0.01 0 -0.12 rpy=0 0 0 -> xyz=0.002 0.02 -0.16 rpy=0 0 0
- joint motor_front_left_leg: limit lower=-2.17 upper=0.97 effort=100.0 velocity=0.5 -> lower=-1.57 upper=1.57 effort=100.0 velocity=0.5
- joint motor_front_right_leg: limit lower=-2.17 upper=0.97 effort=100.0 velocity=0.5 -> lower=-1.57 upper=1.57 effort=100.0 velocity=0.5; origin xyz=0 0.052 0 rpy=0 0 0 -> xyz=0 0.042 0 rpy=0 0 0
- joint motor_rear_left_leg: limit lower=-2.17 upper=0.97 effort=100.0 velocity=0.5 -> lower=-1.57 upper=1.57 effort=100.0 velocity=0.5
- joint motor_rear_right_leg: limit lower=-2.17 upper=0.97 effort=100.0 velocity=0.5 -> lower=-1.57 upper=1.57 effort=100.0 velocity=0.5; origin xyz=0 0.052 0 rpy=0 0 0 -> xyz=0 0.042 0 rpy=0 0 0

Commit message: * mark II: partial design

File: rex_gym/util/pybullet_data/assets/urdf/rex_arm.urdf (robot description, URDF)
Before this commit: robot rex_full, 31 links, 30 joints
Links:
- added link arm_section_1_ext, mass 0; collision cylinder length=0.05 radius=0.02; visual mesh filename=meshes/section_1.obj
- added link arm_section_4_ext, mass 0; collision cylinder length=0.05 radius=0.02; visual mesh filename=meshes/section_4.obj
- link arm_fixed_tip: mass 0.05 -> 0
- link arm_long_U: mass 1. -> 0
- link arm_moving_tip: mass 0.05 -> 0
- link arm_section_1: mass 0.2 -> 0
- link arm_section_2: mass 0.2 -> 0
- link arm_section_3: mass 0.2 -> 0
- link arm_section_4: mass 0.2 -> 0; geometry collision cylinder length=0.05 radius=0.02; visual mesh filename=meshes/section_2.obj
- link arm_section_5: mass 0.2 -> 0
Joints:
- added joint arm_1_ext: type fixed, parent arm_section_1, child arm_section_1_ext, origin xyz=0.048 0 0 rpy=0 1.5707963267949 0, axis 0 0 1
- added joint motor_arm_m7: type revolute, parent arm_section_4_ext, child arm_section_5, origin xyz=0 0 0 rpy=0 0 0, axis 0 0 -1, limit lower=-0.436 upper=1.5 effort=100.0 velocity=0.7
- joint arm_t7f: origin xyz=0 -0.11 0 rpy=-1.5707963267949 0 0 -> xyz=0 0 0 rpy=0 0 0; parent arm_section_4 -> arm_section_4_ext
- joint motor_arm_m1: limit lower=-1.5 upper=1.5 effort=100.0 velocity=0.7 -> lower=-4.71 upper=1.57 effort=100.0 velocity=0.5; origin xyz=-0.03 0 0.0327993216120967 rpy=0 0 0 -> xyz=-0.05 -0.005 0.0327993216120967 rpy=0 0 0
- joint motor_arm_m2: limit lower=-1.5 upper=1.5 effort=100.0 velocity=0.7 -> lower=-1.57 upper=1.57 effort=100.0 velocity=0.5
- joint motor_arm_m3: limit lower=-1.5 upper=1.5 effort=100.0 velocity=0.7 -> lower=-1.57 upper=1.57 effort=100.0 velocity=0.5; origin xyz=0.054 0 0 rpy=0 0 0 -> xyz=0.1 0 0 rpy=0 0 0
- joint motor_arm_m4: limit lower=-1.5 upper=1.5 effort=100.0 velocity=0.7 -> lower=-3.14 upper=3.14 effort=100.0 velocity=0.5
- joint motor_arm_m5: axis 0 0 1 -> 1 0 0; limit lower=-1.5 upper=1.5 effort=100.0 velocity=0.7 -> lower=-1.57 upper=1.57 effort=100.0 velocity=0.5; origin xyz=0 -0.048 0 rpy=0 -1.5707963267949 0 -> xyz=0 -0.048 0 rpy=-1.57 0 3.14
- joint motor_arm_m6: axis 0 0 -1 -> 0 1 0; child arm_section_5 -> arm_section_4_ext; limit lower=-1.3 upper=.2 effort=100.0 velocity=0.7 -> lower=-1.57 upper=1.57 effort=100.0 velocity=0.5; origin xyz=0 -0.058 0 rpy=0 -1.5707963267949 0 -> xyz=0 0 0.097 rpy=-1.57 0 0
