Commit message: * update rex.urdf: update leg link masses. * turn env: minor bugfix.

File: rex_gym/util/pybullet_data/assets/urdf/rex.urdf (robot description, URDF)
Before this commit: robot rex, 23 links, 22 joints
Links:
- link front_left_leg_link_cover: mass None -> 1
- link front_right_leg_link_cover: mass None -> 1
- link rear_left_leg_link_cover: mass None -> 1
- link rear_right_leg_link_cover: mass None -> 1

Commit message: v0.1.0

File: rex_gym/util/pybullet_data/assets/urdf/rex.urdf (robot description, URDF)
Before this commit: robot rex, 23 links, 22 joints
Links:
- link base_link: mass 2.80 -> 1.20
- link chassis_front_link: mass 0.20 -> 0.05
- link chassis_rear_link: mass 0.20 -> 0.05
- link front_left_leg_link: mass 0.15 -> 0.1
- link front_left_leg_link_cover: mass 1 -> 0.5
- link front_left_toe_link: mass 0.05 -> 0.005; geometry collision mesh filename=stl/foot.stl scale=0.001 0.001 0.001; visual mesh filename=stl/foot.stl scale=0.001 0.001 0.001
- link front_right_leg_link: mass 0.15 -> 0.1
- link front_right_leg_link_cover: mass 1 -> 0.5
- link front_right_toe_link: mass 0.05 -> 0.005; geometry collision mesh filename=stl/foot.stl scale=0.001 0.001 0.001; visual mesh filename=stl/foot.stl scale=0.001 0.001 0.001
- link rear_left_leg_link: mass 0.15 -> 0.10
- link rear_left_leg_link_cover: mass 1 -> 0.5
- link rear_left_toe_link: mass 0.05 -> 0.005; geometry collision mesh filename=stl/foot.stl scale=0.001 0.001 0.001; visual mesh filename=stl/foot.stl scale=0.001 0.001 0.001
- link rear_right_leg_link: mass 0.15 -> 0.10
- link rear_right_leg_link_cover: mass 1 -> 0.5
- link rear_right_toe_link: mass 0.05 -> 0.005; geometry collision mesh filename=stl/foot.stl scale=0.001 0.001 0.001; visual mesh filename=stl/foot.stl scale=0.001 0.001 0.001
Joints:
- joint foot_motor_front_left: limit lower=-0.1 upper=2.59 effort=1000.0 velocity=0.5 -> lower=-0.1 upper=2.59 effort=100.0 velocity=0.5
- joint foot_motor_front_right: limit lower=-0.1 upper=2.59 effort=1000.0 velocity=0.5 -> lower=-0.1 upper=2.59 effort=100.0 velocity=0.5
- joint foot_motor_rear_left: limit lower=-0.1 upper=2.59 effort=1000.0 velocity=0.5 -> lower=-0.1 upper=2.59 effort=100.0 velocity=0.5
- joint foot_motor_rear_right: limit lower=-0.1 upper=2.59 effort=1000.0 velocity=0.5 -> lower=-0.1 upper=2.59 effort=100.0 velocity=0.5
- joint motor_front_left_leg: limit lower=-2.666 upper=1.548 effort=1000.0 velocity=0.5 -> lower=-2.17 upper=0.97 effort=100.0 velocity=0.5
- joint motor_front_left_shoulder: limit lower=-0.548 upper=0.548 effort=1000.0 velocity=0.7 -> lower=-1.0 upper=1.0 effort=100.0 velocity=0.7
- joint motor_front_right_leg: limit lower=-2.666 upper=1.548 effort=1000.0 velocity=0.5 -> lower=-2.17 upper=0.97 effort=100.0 velocity=0.5
- joint motor_front_right_shoulder: limit lower=-0.548 upper=0.548 effort=1000.0 velocity=0.7 -> lower=-1.0 upper=1.0 effort=100.0 velocity=0.7
- joint motor_rear_left_leg: limit lower=-2.666 upper=1.548 effort=1000.0 velocity=0.5 -> lower=-2.17 upper=0.97 effort=100.0 velocity=0.5
- joint motor_rear_left_shoulder: limit lower=-0.548 upper=0.548 effort=1000.0 velocity=0.7 -> lower=-1.0 upper=1.0 effort=100.0 velocity=0.7
- joint motor_rear_right_leg: limit lower=-2.666 upper=1.548 effort=1000.0 velocity=0.5 -> lower=-2.17 upper=0.97 effort=100.0 velocity=0.5
- joint motor_rear_right_shoulder: limit lower=-0.548 upper=0.548 effort=1000.0 velocity=0.7 -> lower=-1.0 upper=1.0 effort=100.0 velocity=0.7

Commit message: * proper URDF and STL files

File: rex_gym/util/pybullet_data/assets/urdf/rex.urdf (robot description, URDF)
Before this commit: robot rex, 23 links, 22 joints
Links:
- removed link front_left_leg_link_cover
- removed link front_right_leg_link_cover
- removed link rear_left_leg_link_cover
- removed link rear_right_leg_link_cover
- link base_link: mass 1.20 -> 12; geometry collision mesh filename=stl/mainbody.stl scale=0.001 0.001 0.001; visual mesh filename=stl/mainbody.stl scale=0.001 0.001 0.001
- link chassis_front_link: mass 0.05 -> 0.5; geometry collision mesh filename=stl/frontpart.stl scale=0.001 0.001 0.001; visual mesh filename=stl/frontpart.stl scale=0.001 0.001 0.001
- link chassis_rear_link: mass 0.05 -> 0.5; geometry collision mesh filename=stl/backpart.stl scale=0.001 0.001 0.001; visual mesh filename=stl/backpart.stl scale=0.001 0.001 0.001
- link front_left_foot_link: mass 0.1 -> 0.25; geometry collision mesh filename=stl/lower_leg_solid.stl scale=0.001 0.001 0.001; visual mesh filename=stl/lower_leg_solid.stl scale=0.001 0.001 0.001
- link front_left_leg_link: mass 0.1 -> 1.5; geometry collision mesh filename=stl/upper_leg.stl scale=0.001 0.001 0.001; visual mesh filename=stl/upper_leg.stl scale=0.001 0.001 0.001
- link front_left_shoulder_link: mass 0.10 -> 1; geometry collision mesh filename=stl/shoulder.stl scale=0.001 0.001 0.001; visual mesh filename=stl/shoulder.stl scale=0.001 0.001 0.001
- link front_left_toe_link: mass 0.005 -> 0.01
- link front_right_foot_link: mass 0.1 -> 0.25; geometry collision mesh filename=stl/lower_leg_solid.stl scale=0.001 0.001 0.001; visual mesh filename=stl/lower_leg_solid.stl scale=0.001 0.001 0.001
- link front_right_leg_link: mass 0.1 -> 1.5; geometry collision mesh filename=stl/upper_leg.stl scale=0.001 0.001 0.001; visual mesh filename=stl/upper_leg.stl scale=0.001 0.001 0.001
- link front_right_shoulder_link: mass 0.10 -> 1; geometry collision mesh filename=stl/shoulder.stl scale=0.001 0.001 0.001; visual mesh filename=stl/shoulder.stl scale=0.001 0.001 0.001
- link front_right_toe_link: mass 0.005 -> 0.01
- link rear_left_foot_link: mass 0.1 -> 0.25; geometry collision mesh filename=stl/lower_leg_solid.stl scale=0.001 0.001 0.001; visual mesh filename=stl/lower_leg_solid.stl scale=0.001 0.001 0.001
- link rear_left_leg_link: mass 0.10 -> 1.5; geometry collision mesh filename=stl/upper_leg.stl scale=0.001 0.001 0.001; visual mesh filename=stl/upper_leg.stl scale=0.001 0.001 0.001
- link rear_left_shoulder_link: mass 0.10 -> 1; geometry collision mesh filename=stl/shoulder.stl scale=0.001 0.001 0.001; visual mesh filename=stl/shoulder.stl scale=0.001 0.001 0.001
- link rear_left_toe_link: mass 0.005 -> 0.01
- link rear_right_foot_link: mass 0.1 -> 0.25; geometry collision mesh filename=stl/lower_leg_solid.stl scale=0.001 0.001 0.001; visual mesh filename=stl/lower_leg_solid.stl scale=0.001 0.001 0.001
- link rear_right_leg_link: mass 0.10 -> 1.5; geometry collision mesh filename=stl/upper_leg.stl scale=0.001 0.001 0.001; visual mesh filename=stl/upper_leg.stl scale=0.001 0.001 0.001
- link rear_right_shoulder_link: mass 0.10 -> 1; geometry collision mesh filename=stl/shoulder.stl scale=0.001 0.001 0.001; visual mesh filename=stl/shoulder.stl scale=0.001 0.001 0.001
- link rear_right_toe_link: mass 0.005 -> 0.01
Joints:
- removed joint front_left_leg_cover_joint
- removed joint front_left_toe
- removed joint front_right_leg_cover_joint
- removed joint front_right_toe
- removed joint rear_left_leg_cover_joint
- removed joint rear_left_toe
- removed joint rear_right_leg_cover_joint
- removed joint rear_right_toe
- added joint toe_joint_front_left: type fixed, parent front_left_foot_link, child front_left_toe_link, origin xyz=0 -0.0098 -0.16
- added joint toe_joint_front_right: type fixed, parent front_right_foot_link, child front_right_toe_link, origin xyz=0 -0.0098 -0.16
- added joint toe_joint_rear_left: type fixed, parent rear_left_foot_link, child rear_left_toe_link, origin xyz=0 -0.0098 -0.16
- added joint toe_joint_rear_right: type fixed, parent rear_right_foot_link, child rear_right_toe_link, origin xyz=0 -0.0098 -0.16
- joint chassis_base_front: origin (none) -> xyz=-0.042 -0.055 -0.01 rpy=0 0 0
- joint chassis_base_rear: origin (none) -> xyz=0.05 0 -0.038 rpy=0 0 0
- joint foot_motor_front_left: limit lower=-3.14 upper=3.14 effort=100.0 velocity=0.5 -> lower=-3.14 upper=3.14 effort=100.0 velocity=100; origin xyz=0.002 -0.02 -0.16 rpy=0 0 0 -> xyz=0 -0.047 -0.16 rpy=0 0 0
- joint foot_motor_front_right: limit lower=-3.14 upper=3.14 effort=100.0 velocity=0.5 -> lower=-3.14 upper=3.14 effort=100.0 velocity=100; origin xyz=0.002 0.02 -0.16 rpy=0 0 0 -> xyz=0 0.047 -0.16 rpy=0 0 0
- joint foot_motor_rear_left: limit lower=-3.14 upper=3.14 effort=100.0 velocity=0.5 -> lower=-3.14 upper=3.14 effort=100.0 velocity=100; origin xyz=0.002 -0.02 -0.16 rpy=0 0 0 -> xyz=0 -0.047 -0.16 rpy=0 0 0
- joint foot_motor_rear_right: limit lower=-3.14 upper=3.14 effort=100.0 velocity=0.5 -> lower=-3.14 upper=3.14 effort=100.0 velocity=100; origin xyz=0.002 0.02 -0.16 rpy=0 0 0 -> xyz=0 0.047 -0.16 rpy=0 0 0
- joint motor_front_left_leg: limit lower=-1.57 upper=1.57 effort=100.0 velocity=0.5 -> lower=-1.57 upper=1.57 effort=100.0 velocity=100; origin xyz=0 -0.052 0 rpy=0 0 0 -> xyz=0 -0.017 0 rpy=0 0 0
- joint motor_front_left_shoulder: limit lower=-1.0 upper=1.0 effort=100.0 velocity=0.7 -> lower=-1.0 upper=1.0 effort=100.0 velocity=100; origin xyz=-0.093 -0.036 0 rpy=0 0 0 -> xyz=-0.095 -0.035 0 rpy=0 0 0
- joint motor_front_right_leg: limit lower=-1.57 upper=1.57 effort=100.0 velocity=0.5 -> lower=-1.57 upper=1.57 effort=100.0 velocity=100; origin xyz=0 0.042 0 rpy=0 0 0 -> xyz=0 0.017 0 rpy=0 0 0
- joint motor_front_right_shoulder: limit lower=-1.0 upper=1.0 effort=100.0 velocity=0.7 -> lower=-1.0 upper=1.0 effort=100.0 velocity=100; origin xyz=-0.093 0.036 0 rpy=0 0 0 -> xyz=-0.095 0.035 0 rpy=0 0 0
- joint motor_rear_left_leg: limit lower=-1.57 upper=1.57 effort=100.0 velocity=0.5 -> lower=-1.57 upper=1.57 effort=100.0 velocity=100; origin xyz=0 -0.052 0 rpy=0 0 0 -> xyz=0 -0.017 0 rpy=0 0 0
- joint motor_rear_left_shoulder: limit lower=-1.0 upper=1.0 effort=100.0 velocity=0.7 -> lower=-1.0 upper=1.0 effort=100.0 velocity=100; origin xyz=0.093 -0.036 0 rpy=0 0 0 -> xyz=0.09 -0.035 0 rpy=0 0 0
- joint motor_rear_right_leg: limit lower=-1.57 upper=1.57 effort=100.0 velocity=0.5 -> lower=-1.57 upper=1.57 effort=100.0 velocity=100; origin xyz=0 0.042 0 rpy=0 0 0 -> xyz=0 0.017 0 rpy=0 0 0
- joint motor_rear_right_shoulder: limit lower=-1.0 upper=1.0 effort=100.0 velocity=0.7 -> lower=-1.0 upper=1.0 effort=100.0 velocity=100; origin xyz=0.093 0.036 0 rpy=0 0 0 -> xyz=0.09 0.035 0 rpy=0 0 0

File: rex_gym/util/pybullet_data/assets/urdf/rex_arm.urdf (robot description, URDF)
Before this commit: robot rex_full, 33 links, 32 joints
Joints:
- removed joint front_left_toe
- removed joint front_right_toe
- removed joint rear_left_toe
- removed joint rear_right_toe
- added joint toe_joint_front_left: type fixed, parent front_left_foot_link, child front_left_toe_link, origin xyz=0 0 -0.115
- added joint toe_joint_front_right: type fixed, parent front_right_foot_link, child front_right_toe_link, origin xyz=0 0 -0.115
- added joint toe_joint_rear_left: type fixed, parent rear_left_foot_link, child rear_left_toe_link, origin xyz=0 0 -0.115
- added joint toe_joint_rear_right: type fixed, parent rear_right_foot_link, child rear_right_toe_link, origin xyz=0 0 -0.115
